Commit message: replaced RealMan arm with 7-dof model, also adjusted installation location. Left-arm only

File: urdf/PatrolRobot.urdf (robot description, URDF)
Before this commit: robot PatrolRobot, 27 links, 26 joints
Links:
- added link Link7, mass 0.14433; collision mesh filename=package://patrolrobot/meshes/Link7.STL; visual mesh filename=package://patrolrobot/meshes/Link7.STL
- link Link1: geometry collision mesh filename=package://patrolrobot/meshes/Link1.STL; visual mesh filename=package://patrolrobot/meshes/Link1.STL
- link Link2: mass 0.86418 -> 0.43285; geometry collision mesh filename=package://patrolrobot/meshes/Link2.STL; visual mesh filename=package://patrolrobot/meshes/Link2.STL
- link Link3: mass 0.28965 -> 0.43132; geometry collision mesh filename=package://patrolrobot/meshes/Link3.STL; visual mesh filename=package://patrolrobot/meshes/Link3.STL
- link Link4: mass 0.23942 -> 0.28963; geometry collision mesh filename=package://patrolrobot/meshes/Link4.STL; visual mesh filename=package://patrolrobot/meshes/Link4.STL
- link Link5: mass 0.21879 -> 0.23941; geometry collision mesh filename=package://patrolrobot/meshes/Link5.STL; visual mesh filename=package://patrolrobot/meshes/Link5.STL
- link Link6: mass 0.065035 -> 0.21879; geometry collision mesh filename=package://patrolrobot/meshes/Link6.STL; visual mesh filename=package://patrolrobot/meshes/Link6.STL
- link base_link: geometry collision mesh filename=package://patrolrobot/meshes/base_link.STL; visual mesh filename=package://patrolrobot/meshes/base_link.STL
Joints:
- added joint joint7: type revolute, parent Link6, child Link7, origin xyz=0 0 0.1725 rpy=0 0 0, axis 0 0 1, limit lower=-6.283 upper=6.283 effort=10 velocity=1
- joint base_link: origin xyz=-0.02 0.175 0.5 rpy=-1.5708 0 0 -> xyz=-0.02 0.0175 0.5 rpy=-1.5708 -1.57 0
- joint joint1: axis 0 0 1 -> 0 -1 0; origin xyz=0 0 0.2405 rpy=0 0 0 -> xyz=0 0 0.2405 rpy=-1.5708 0 0
- joint joint2: axis 0 0 1 -> 0 1 0; origin xyz=0 0 0 rpy=1.5708 -1.5708 0 -> xyz=0 0 0 rpy=1.5708 0 0
- joint joint3: axis 0 0 1 -> 0 -1 0; limit lower=-2.356 upper=2.356 effort=30 velocity=1 -> lower=-3.107 upper=3.107 effort=10 velocity=1; origin xyz=0.256 0 0 rpy=0 0 1.5708 -> xyz=0 0 0.256 rpy=-1.5708 0 0
- joint joint4: axis 0 0 1 -> 0 1 0; limit lower=-3.107 upper=3.107 effort=10 velocity=1 -> lower=-2.356 upper=2.356 effort=30 velocity=1; origin xyz=0 -0.21 0 rpy=1.5708 0 0 -> xyz=0 0 0 rpy=1.5708 0 0
- joint joint5: axis 0 0 1 -> 0 -1 0; limit lower=-2.234 upper=2.234 effort=10 velocity=1 -> lower=-3.107 upper=3.107 effort=10 velocity=1; origin xyz=0 0 0 rpy=-1.5708 0 0 -> xyz=0 0 0.21 rpy=-1.5708 0 0
- joint joint6: axis 0 0 1 -> 0 1 0; limit lower=-6.283 upper=6.283 effort=10 velocity=1 -> lower=-2.234 upper=2.234 effort=10 velocity=1; origin xyz=0 -0.144 0 rpy=1.5708 0 0 -> xyz=0 0 0 rpy=1.5708 0 0

Commit message: added right arm to the robot model; next step is to add convex hulls and collision checks

File: urdf/PatrolRobot.urdf (robot description, URDF)
Before this commit: robot PatrolRobot, 28 links, 27 joints
Links:
- removed link Link1
- removed link Link2
- removed link Link3
- removed link Link4
- removed link Link5
- removed link Link6
- removed link Link7
- removed link base_link
- removed link relbowpitch
- removed link righthand
- removed link rshoulderpitch
- removed link rshoulderroll
- removed link rshoulderyaw
- removed link rwristpitch
- removed link rwristroll
- added link LArm0, mass 0.84108; collision mesh filename=package://patrolrobot/meshes/LArm0.STL; visual mesh filename=package://patrolrobot/meshes/LArm0.STL
- added link LArm1, mass 0.59356; collision mesh filename=package://patrolrobot/meshes/LArm1.STL; visual mesh filename=package://patrolrobot/meshes/LArm1.STL
- added link LArm2, mass 0.43285; collision mesh filename=package://patrolrobot/meshes/LArm2.STL; visual mesh filename=package://patrolrobot/meshes/LArm2.STL
- added link LArm3, mass 0.43132; collision mesh filename=package://patrolrobot/meshes/LArm3.STL; visual mesh filename=package://patrolrobot/meshes/LArm3.STL
- added link LArm4, mass 0.28963; collision mesh filename=package://patrolrobot/meshes/LArm4.STL; visual mesh filename=package://patrolrobot/meshes/LArm4.STL
- added link LArm5, mass 0.23941; collision mesh filename=package://patrolrobot/meshes/LArm5.STL; visual mesh filename=package://patrolrobot/meshes/LArm5.STL
- added link LArm6, mass 0.21879; collision mesh filename=package://patrolrobot/meshes/LArm6.STL; visual mesh filename=package://patrolrobot/meshes/LArm6.STL
- added link LArm7, mass 0.14433; collision mesh filename=package://patrolrobot/meshes/LArm7.STL; visual mesh filename=package://patrolrobot/meshes/LArm7.STL
- added link RArm0, mass 0.84108; collision mesh filename=package://patrolrobot/meshes/RArm0.STL; visual mesh filename=package://patrolrobot/meshes/RArm0.STL
- added link RArm1, mass 0.59356; collision mesh filename=package://patrolrobot/meshes/RArm1.STL; visual mesh filename=package://patrolrobot/meshes/RArm1.STL
- added link RArm2, mass 0.43285; collision mesh filename=package://patrolrobot/meshes/RArm2.STL; visual mesh filename=package://patrolrobot/meshes/RArm2.STL
- added link RArm3, mass 0.43132; collision mesh filename=package://patrolrobot/meshes/RArm3.STL; visual mesh filename=package://patrolrobot/meshes/RArm3.STL
- added link RArm4, mass 0.28963; collision mesh filename=package://patrolrobot/meshes/RArm4.STL; visual mesh filename=package://patrolrobot/meshes/RArm4.STL
- added link RArm5, mass 0.23941; collision mesh filename=package://patrolrobot/meshes/RArm5.STL; visual mesh filename=package://patrolrobot/meshes/RArm5.STL
- added link RArm6, mass 0.21879; collision mesh filename=package://patrolrobot/meshes/RArm6.STL; visual mesh filename=package://patrolrobot/meshes/RArm6.STL
- added link RArm7, mass 0.14433; collision mesh filename=package://patrolrobot/meshes/RArm7.STL; visual mesh filename=package://patrolrobot/meshes/RArm7.STL
Joints:
- removed joint base_link
- removed joint joint1
- removed joint joint2
- removed joint joint3
- removed joint joint4
- removed joint joint5
- removed joint joint6
- removed joint joint7
- removed joint relbowpitch
- removed joint righthand
- removed joint rshoulderpitch
- removed joint rshoulderroll
- removed joint rshoulderyaw
- removed joint rwristpitch
- removed joint rwristroll
- added joint LArm0: type fixed, parent torso, child LArm0, origin xyz=-0.02 0.0175 0.5 rpy=-1.5708 1.57 0
- added joint LArm1: type revolute, parent LArm0, child LArm1, origin xyz=0 0 0.2405 rpy=-1.5708 0 0, axis 0 -1 0, limit lower=-3.107 upper=3.107 effort=60 velocity=1
- added joint LArm2: type revolute, parent LArm1, child LArm2, origin xyz=0 0 0 rpy=1.5708 0 0, axis 0 1 0, limit lower=-2.269 upper=2.269 effort=60 velocity=1
- added joint LArm3: type revolute, parent LArm2, child LArm3, origin xyz=0 0 0.256 rpy=-1.5708 0 0, axis 0 -1 0, limit lower=-3.107 upper=3.107 effort=10 velocity=1
- added joint LArm4: type revolute, parent LArm3, child LArm4, origin xyz=0 0 0 rpy=1.5708 0 0, axis 0 1 0, limit lower=-2.356 upper=2.356 effort=30 velocity=1
- added joint LArm5: type revolute, parent LArm4, child LArm5, origin xyz=0 0 0.21 rpy=-1.5708 0 0, axis 0 -1 0, limit lower=-3.107 upper=3.107 effort=10 velocity=1
- added joint LArm6: type revolute, parent LArm5, child LArm6, origin xyz=0 0 0 rpy=1.5708 0 0, axis 0 1 0, limit lower=-2.234 upper=2.234 effort=10 velocity=1
- added joint LArm7: type revolute, parent LArm6, child LArm7, origin xyz=0 0 0.1725 rpy=0 0 0, axis 0 0 1, limit lower=-6.283 upper=6.283 effort=10 velocity=1
- added joint RArm0: type fixed, parent torso, child RArm0, origin xyz=-0.02 -0.0175 0.5 rpy=1.5708 1.57 0
- added joint RArm1: type revolute, parent RArm0, child RArm1, origin xyz=0 0 0.2405 rpy=-1.5708 0 0, axis 0 -1 0, limit lower=-3.107 upper=3.107 effort=60 velocity=1
- added joint RArm2: type revolute, parent RArm1, child RArm2, origin xyz=0 0 0 rpy=1.5708 0 0, axis 0 1 0, limit lower=-2.269 upper=2.269 effort=60 velocity=1
- added joint RArm3: type revolute, parent RArm2, child RArm3, origin xyz=0 0 0.256 rpy=-1.5708 0 0, axis 0 -1 0, limit lower=-3.107 upper=3.107 effort=10 velocity=1
- added joint RArm4: type revolute, parent RArm3, child RArm4, origin xyz=0 0 0 rpy=1.5708 0 0, axis 0 1 0, limit lower=-2.356 upper=2.356 effort=30 velocity=1
- added joint RArm5: type revolute, parent RArm4, child RArm5, origin xyz=0 0 0.21 rpy=-1.5708 0 0, axis 0 -1 0, limit lower=-3.107 upper=3.107 effort=10 velocity=1
- added joint RArm6: type revolute, parent RArm5, child RArm6, origin xyz=0 0 0 rpy=1.5708 0 0, axis 0 1 0, limit lower=-2.234 upper=2.234 effort=10 velocity=1
- added joint RArm7: type revolute, parent RArm6, child RArm7, origin xyz=0 0 0.1725 rpy=0 0 0, axis 0 0 1, limit lower=-6.283 upper=6.283 effort=10 velocity=1
